File: hot-plate-kicad_final.kicad_sch (KiCad schematic)
At the start: 29 parts, among them J1 IEC - 60320, M1 Fan, Q1 Q_NPN_BCE, Q2 Q_NPN_BCE, SW1 SW_DPST_x2, U2 MAX36675

Commit message: Final Schematic of the Electrical Part
Other:
- note removed: "connect to the pin of arduino"
- note removed: "goes to arduino"
Changed lines of the file:
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@@
-    (effects (font (size 1.27 1.27)) (justify left bottom))
-  )
-  (text "goes to arduino\n" (at 78.74 85.09 0)
-    (effects (font (size 1.27 1.27)) (justify left bottom))
-  )
-  (text "connect to the pin of arduino\n" (at 96.52 40.64 0)
     (effects (font (size 1.27 1.27)) (justify left bottom))
   )
@@
       (effects (font (size 1.27 1.27)) hide)
     )
-    (property "Value" "MAX36675" (at 92.71 20.32 90)
-      (effects (font (size 1.27 1.27)))
-    )
+    (property "Value" "MAX36675" (at 80.01 17.78 90)
+      (effects (font (size 1.27 1.27)))
+    )
